Commit message: feat: 使用 ros2-control 让小车在 Gazebo 中运动

File: src/robot_describes/urdf/ackermann_car.urdf.xacro (robot description, xacro)
@@ -1,179 +1,44 @@
 <?xml version="1.0"?>
 <robot xmlns:xacro="http://www.ros.org/wiki/xacro" name="xbot">
-  <!-- ==================== 参数 ==================== -->
-  <xacro:property name="scale"   value="1"/>
-  <!-- yu7 参数 -->
-  <!-- 轮子半径 -->
-  <xacro:property name="wheel_radius" value="${0.3625 * scale}"/>
-  <!-- 轮子宽度 -->
-  <xacro:property name="wheel_width" value="${0.242 * scale}"/>
-  <!-- 车身宽度 -->
-  <xacro:property name="base_width"   value="${1.95 * scale}"/>
-  <!-- 车身长度 -->
-  <xacro:property name="base_length"   value="${4.7 * scale}"/>
-  <!-- 车身高度 -->
-  <xacro:property name="base_height"   value="${1.3 * scale}"/>
-  <!-- 车身 z 轴距离 -->
-  <xacro:property name="base_z"   value="${0.24 * scale}"/>
-  <!-- 车身重量 -->
-  <xacro:property name="base_mass"   value="${1500 * scale}"/>
-  <!-- 轮子重量 -->
-  <xacro:property name="wheel_mass"   value="${50 * scale}"/>
-  <!-- ==================== 虚拟根链接 ==================== -->
-  <link name="base_footprint"/>
-  <joint name="base_footprint_joint" type="fixed">
-    <parent link="base_footprint"/>
-    <child link="base_link"/>
-    <origin xyz="0 0 0" rpy="0 0 0"/>
-  </joint>
-  <!-- ==================== 车身 ==================== -->
-  <link name="base_link">
-    <visual>
-      <geometry>
-        <mesh filename="package://robot_describes/model/yu7_body.glb" scale="${scale} ${scale} ${scale}"/>
-      </geometry>
-    </visual>
-    <collision>
-      <geometry>
-        <box size="${base_length} ${base_width} ${base_height}"/>
-      </geometry>
-      <origin xyz="0 0 ${base_height / 2 + base_z}"/>
-    </collision>
-    <inertial>
-      <mass value="${base_mass}" />
-      <origin xyz="0 0 ${base_height / 2 + base_z}"/>
-      <inertia ixx="${(base_mass/12) * (base_width*base_width + base_height*base_height)}" ixy="0.0" ixz="0.0" iyy="${(base_mass/12) * (base_length*base_length + base_height*base_height)}" iyz="0.0" izz="${(base_mass/12) * (base_length*base_length + base_width*base_width)}" />
-    </inertial>
-  </link>
-  <!-- ==================== 前左轮连杆 ==================== -->
-  <link name="left_wheel_steering">
-    <inertial>
-      <mass value="0.1"/>
-      <inertia ixx="0.001" ixy="0.0" ixz="0.0" iyy="0.001" iyz="0.0" izz="0.002" />
-    </inertial>
-  </link>
-  <joint name="left_wheel_steering_joint" type="revolute">
-    <origin xyz="${-1.436 * scale} ${-0.8554 * scale} ${0.4034 * scale}"/>
-    <parent link="base_link" />
-    <child link="left_wheel_steering" />
-    <axis xyz="0 0 1" />
-    <dynamics damping="0.2" />
-    <limit effort="1000.0" lower="-1.57" upper="1.57" velocity="30"/>
-  </joint>
-  <!-- ==================== 前右轮连杆 ==================== -->
-  <link name="right_wheel_steering">
-    <inertial>
-      <mass value="0.1"/>
-      <inertia ixx="0.001" ixy="0.0" ixz="0.0" iyy="0.001" iyz="0.0" izz="0.002" />
-    </inertial>
-  </link>
-  <joint name="right_wheel_steering_joint" type="revolute">
-    <origin xyz="${-1.436 * scale} ${0.8554 * scale} ${0.4034 * scale}"/>
-    <parent link="base_link" />
-    <child link="right_wheel_steering" />
-    <axis xyz="0 0 1" />
-    <dynamics damping="0.2" />
-    <limit effort="1000.0" lower="-1.57" upper="1.57" velocity="30"/>
-  </joint>
-  <!-- ==================== 前左轮 ==================== -->
-  <link name="front_left_wheel">
-    <visual>
-      <geometry>
-        <mesh filename="package://robot_describes/model/yu7_wheel.glb" scale="${scale} ${scale} ${scale}"/>
-      </geometry>
-    </visual>
-    <collision>
-      <geometry>
-        <cylinder radius="${wheel_radius}" length="${wheel_width}"/>
-      </geometry>
-      <origin rpy="1.5708 0 0"/>
-    </collision>
-    <inertial>
-      <origin rpy="1.5708 0 0"/>
-      <mass value="${wheel_mass}" />
-      <inertia ixx="${(wheel_mass/12) * (3*wheel_radius*wheel_radius + wheel_width*wheel_width)}" ixy="0" ixz="0" iyy="${(wheel_mass/12) * (3*wheel_radius*wheel_radius + wheel_width*wheel_width)}" iyz="0" izz="${(wheel_mass/2) * (wheel_radius*wheel_radius)}" />
-    </inertial>
-  </link>
-  <joint name="front_left_wheel_joint" type="continuous">
-    <parent link="left_wheel_steering"/>
-    <child link="front_left_wheel"/>
-    <origin xyz="0 0 0"/>
-    <axis xyz="0 1 0"/>
-  </joint>
-  <!-- ==================== 前右轮 ==================== -->
-  <link name="front_right_wheel">
-    <visual>
-      <geometry>
-        <mesh filename="package://robot_describes/model/yu7_wheel.glb" scale="${scale} ${scale} ${scale}"/>
-      </geometry>
-    </visual>
-    <collision>
-      <geometry>
-        <cylinder radius="${wheel_radius}" length="${wheel_width}"/>
-      </geometry>
-      <origin rpy="1.5708 0 0"/>
-    </collision>
-    <inertial>
-      <origin rpy="1.5708 0 0"/>
-      <mass value="${wheel_mass}" />
-      <inertia ixx="${(wheel_mass/12) * (3*wheel_radius*wheel_radius + wheel_width*wheel_width)}" ixy="0" ixz="0" iyy="${(wheel_mass/12) * (3*wheel_radius*wheel_radius + wheel_width*wheel_width)}" iyz="0" izz="${(wheel_mass/2) * (wheel_radius*wheel_radius)}" />
-    </inertial>
-  </link>
-  <joint name="front_right_wheel_joint" type="continuous">
-    <parent link="right_wheel_steering"/>
-    <child link="front_right_wheel"/>
-    <origin xyz="0 0 0" rpy="0 0 3.1415926"/>
-    <axis xyz="0 -1 0"/>
-  </joint>
-  <!-- ==================== 后左轮 ==================== -->
-  <link name="rear_left_wheel">
-    <visual>
-      <geometry>
-        <mesh filename="package://robot_describes/model/yu7_wheel.glb" scale="${scale} ${scale} ${scale}"/>
-      </geometry>
-    </visual>
-    <collision>
-      <geometry>
-        <cylinder radius="${wheel_radius}" length="${wheel_width}"/>
-      </geometry>
-      <origin rpy="1.5708 0 0"/>
-    </collision>
-    <inertial>
-      <origin rpy="1.5708 0 0"/>
-      <mass value="${wheel_mass}" />
-      <inertia ixx="${(wheel_mass/12) * (3*wheel_radius*wheel_radius + wheel_width*wheel_width)}" ixy="0" ixz="0" iyy="${(wheel_mass/12) * (3*wheel_radius*wheel_radius + wheel_width*wheel_width)}" iyz="0" izz="${(wheel_mass/2) * (wheel_radius*wheel_radius)}" />
-    </inertial>
-  </link>
-  <joint name="rear_left_wheel_joint" type="continuous">
-    <parent link="base_link"/>
-    <child link="rear_left_wheel"/>
-    <origin xyz="${1.402 * scale} ${-0.8736 * scale} ${0.4034 * scale}"/>
-    <axis xyz="0 1 0"/>
-  </joint>
-  <!-- ==================== 后右轮 ==================== -->
-  <link name="rear_right_wheel">
-    <visual>
-      <!-- <origin rpy="0 0 3.1415926"/> -->
-      <geometry>
-        <mesh filename="package://robot_describes/model/yu7_wheel.glb" scale="${scale} ${scale} ${scale}"/>
-      </geometry>
-    </visual>
-    <collision>
-      <geometry>
-        <cylinder radius="${wheel_radius}" length="${wheel_width}"/>
-      </geometry>
-      <origin rpy="1.5708 0 0"/>
-    </collision>
-    <inertial>
-      <origin rpy="1.5708 0 0"/>
-      <mass value="${wheel_mass}" />
-      <inertia ixx="${(wheel_mass/12) * (3*wheel_radius*wheel_radius + wheel_width*wheel_width)}" ixy="0" ixz="0" iyy="${(wheel_mass/12) * (3*wheel_radius*wheel_radius + wheel_width*wheel_width)}" iyz="0" izz="${(wheel_mass/2) * (wheel_radius*wheel_radius)}" />
-    </inertial>
-  </link>
-  <joint name="rear_right_wheel_joint" type="continuous">
-    <parent link="base_link"/>
-    <child link="rear_right_wheel"/>
-    <origin xyz="${1.402 * scale} ${0.8736 * scale} ${0.4034 * scale}" rpy="0 0 3.1415926"/>
-    <axis xyz="0 -1 0"/>
-  </joint>
+  <xacro:include filename="$(find robot_describes)/urdf/ackermann_yu7.xacro"/>
+  <!-- 车身 -->
+  <xacro:yu7 visual_rpy="1.5708 0 0"/>
+  <!-- ros2 control 声明接口 -->
+  <ros2_control name="GazeboSystem" type="system">
+    <hardware>
+      <plugin>gz_ros2_control/GazeboSimSystem</plugin>
+    </hardware>
+    <joint name="rear_left_wheel_joint">
+      <command_interface name="velocity" />
+      <state_interface name="velocity" />
+      <state_interface name="position" />
+    </joint>
+    <joint name="rear_right_wheel_joint">
+      <command_interface name="velocity" />
+      <state_interface name="velocity" />
+      <state_interface name="position" />
+    </joint>
+    <joint name="left_wheel_steering_joint">
+      <command_interface name="position" />
+      <state_interface name="position" />
+    </joint>
+    <joint name="right_wheel_steering_joint">
+      <command_interface name="position" />
+      <state_interface name="position" />
+    </joint>
+    <joint name="front_left_wheel_joint">
+      <state_interface name="position" />
+      <state_interface name="velocity" />
+    </joint>
+    <joint name="front_right_wheel_joint">
+      <state_interface name="position" />
+      <state_interface name="velocity" />
+    </joint>
+  </ros2_control>
+  <!-- gazebo 插件，管理 control manager -->
+  <gazebo>
+    <plugin filename="gz_ros2_control-system" name="gz_ros2_control::GazeboSimROS2ControlPlugin">
+      <parameters>$(find robot_describes)/config/ackermann_drive_controller.yaml</parameters>
+    </plugin>
+  </gazebo>
 </robot>
